Commit message: fixed model loading

File: ros_src/custom_sawyer_description/urdf/custom_sawyer_camera.urdf.xacro (robot description, xacro)
@@ -1,6 +1,6 @@
 <?xml version="1.0" ?>
 <robot name="sawyer" xmlns:xacro="http://www.ros.org/wiki/xacro">
-    <xacro:include filename="$(find custom_sawyer_description)/urdf/camera_2D.xacro"/>
-    <xacro:include filename="$(find custom_sawyer_description)/urdf/camera_2D_gazebo.xacro"/>
+    <!-- <xacro:include filename="$(find custom_sawyer_description)/urdf/camera_2D.xacro"/>
+    <xacro:include filename="$(find custom_sawyer_description)/urdf/camera_2D_gazebo.xacro"/> -->
         <xacro:include filename="$(find custom_sawyer_description)/urdf/kinetic_rgb.urdf.xacro"/>
      <xacro:property name="deg_to_rad" value="0.01745329251994329577"/>
@@ -31,6 +31,10 @@
   </xacro:include>
   </xacro:if>
-    <xacro:kinetic_rgb name="rgbd_camera" parent="base">
-        <origin xyz="0.1 0.0 1.3" rpy="${0.0 * deg_to_rad} ${70.0 * deg_to_rad} ${0.0 * deg_to_rad}"/>
+    <xacro:kinetic_rgb name="rgbd_camera_right" parent="base">
+        <origin xyz="0.8 -0.4 0.5" rpy="${0.0 * deg_to_rad} ${60.0 * deg_to_rad} ${90.0 * deg_to_rad}"/>
+        <origin xyz="0 0 0" rpy="${-90 * deg_to_rad} ${0 * deg_to_rad} ${-90 * deg_to_rad}" />
+    </xacro:kinetic_rgb>
+    <xacro:kinetic_rgb name="rgbd_camera_left" parent="base">
+        <origin xyz="0.8 0.4 0.5" rpy="${0.0 * deg_to_rad} ${60.0 * deg_to_rad} ${-90.0 * deg_to_rad}"/>
         <origin xyz="0 0 0" rpy="${-90 * deg_to_rad} ${0 * deg_to_rad} ${-90 * deg_to_rad}" />
     </xacro:kinetic_rgb>

Commit message: Add new models for banana and coke can, including textures and configuration files

File: ros_src/custom_sawyer_description/urdf/custom_sawyer_camera.urdf.xacro (robot description, xacro)
@@ -21,20 +21,21 @@
     </xacro:include>
   </xacro:if>
-  <!-- <xacro:if value="$(arg electric_gripper)">
+   <xacro:if value="$(arg electric_gripper)">
     <xacro:include filename="$(find sawyer_description)/urdf/sawyer_electric_gripper.urdf.xacro">
       <xacro:arg name="gazebo" value="${gazebo}"/>
     </xacro:include>
-  </xacro:if> -->
-    <xacro:if value="$(arg electric_gripper)">
+  </xacro:if>
+    <!-- <xacro:if value="$(arg electric_gripper)">
   <xacro:include filename="$(find pneumatic_gripper_description)/urdf/pneumatic_gripper.urdf.xacro">
     <xacro:arg name="gazebo" value="${gazebo}"/>
   </xacro:include>
   </xacro:if>
+ -->
     <xacro:kinetic_rgb name="rgbd_camera_right" parent="base">
-        <origin xyz="0.8 -0.4 0.5" rpy="${0.0 * deg_to_rad} ${60.0 * deg_to_rad} ${90.0 * deg_to_rad}"/>
+        <origin xyz="0.55 -0.6 0.5" rpy="${0.0 * deg_to_rad} ${60.0 * deg_to_rad} ${90.0 * deg_to_rad}"/>
         <origin xyz="0 0 0" rpy="${-90 * deg_to_rad} ${0 * deg_to_rad} ${-90 * deg_to_rad}" />
     </xacro:kinetic_rgb>
     <xacro:kinetic_rgb name="rgbd_camera_left" parent="base">
-        <origin xyz="0.8 0.4 0.5" rpy="${0.0 * deg_to_rad} ${60.0 * deg_to_rad} ${-90.0 * deg_to_rad}"/>
+        <origin xyz="0.55 0.6 0.5" rpy="${0.0 * deg_to_rad} ${60.0 * deg_to_rad} ${-90.0 * deg_to_rad}"/>
         <origin xyz="0 0 0" rpy="${-90 * deg_to_rad} ${0 * deg_to_rad} ${-90 * deg_to_rad}" />
     </xacro:kinetic_rgb>

Commit message: Refactor and enhance TossingBot learning and planning modules
- Replaced SumTree with RankBasedReplayBuffer for prioritized experience replay in buffer.py.
- Updated network.py to improve ResidualBlock with clearer comments and structure.
- Enhanced utils.py with normalization for image tensors and improved rotation handling.
- Refined casadi_planner.py to utilize PlannerConfig for better parameter management and added detailed comments.
- Introduced planner_config.py to centralize planning parameters and weights.
- Added auto_grasp.py script for automated grasping with visualization and decision-making logic.
- Updated weights: replaced rotational invariant weights with new auto weights.

File: ros_src/custom_sawyer_description/urdf/custom_sawyer_camera.urdf.xacro (robot description, xacro)
@@ -33,9 +33,9 @@
  -->
     <xacro:kinetic_rgb name="rgbd_camera_right" parent="base">
-        <origin xyz="0.55 -0.6 0.5" rpy="${0.0 * deg_to_rad} ${60.0 * deg_to_rad} ${90.0 * deg_to_rad}"/>
+        <origin xyz="0.55 -0.4 0.35" rpy="${0.0 * deg_to_rad} ${50.0 * deg_to_rad} ${90.0 * deg_to_rad}"/>
         <origin xyz="0 0 0" rpy="${-90 * deg_to_rad} ${0 * deg_to_rad} ${-90 * deg_to_rad}" />
     </xacro:kinetic_rgb>
     <xacro:kinetic_rgb name="rgbd_camera_left" parent="base">
-        <origin xyz="0.55 0.6 0.5" rpy="${0.0 * deg_to_rad} ${60.0 * deg_to_rad} ${-90.0 * deg_to_rad}"/>
+        <origin xyz="0.55 0.4 0.35" rpy="${0.0 * deg_to_rad} ${50.0 * deg_to_rad} ${-90.0 * deg_to_rad}"/>
         <origin xyz="0 0 0" rpy="${-90 * deg_to_rad} ${0 * deg_to_rad} ${-90 * deg_to_rad}" />
     </xacro:kinetic_rgb>

Commit message: Add velocity measurement and tossing functionality
- Implemented `test_velocity_measurement.py` to measure actual velocities during tosses, logging results to a CSV file.
- Created `toss_to_target.py` for inverse tossing experiments, calculating required speeds based on target positions and executing tosses.
- Developed `physics_controller.py` to handle ballistic trajectory calculations, including release parameters and velocity components.
- Introduced `velocity_monitor.py` to track and analyze end-effector and object velocities during tossing, providing detailed analysis and peak velocity data.
- Added an empty `__init__.py` file in the utils module for package initialization.

File: ros_src/custom_sawyer_description/urdf/custom_sawyer_camera.urdf.xacro (robot description, xacro)
@@ -33,9 +33,9 @@
  -->
     <xacro:kinetic_rgb name="rgbd_camera_right" parent="base">
-        <origin xyz="0.55 -0.4 0.35" rpy="${0.0 * deg_to_rad} ${50.0 * deg_to_rad} ${90.0 * deg_to_rad}"/>
+        <origin xyz="0.55 -0.2637 0.35" rpy="${0.0 * deg_to_rad} ${50.0 * deg_to_rad} ${90.0 * deg_to_rad}"/>
         <origin xyz="0 0 0" rpy="${-90 * deg_to_rad} ${0 * deg_to_rad} ${-90 * deg_to_rad}" />
     </xacro:kinetic_rgb>
     <xacro:kinetic_rgb name="rgbd_camera_left" parent="base">
-        <origin xyz="0.55 0.4 0.35" rpy="${0.0 * deg_to_rad} ${50.0 * deg_to_rad} ${-90.0 * deg_to_rad}"/>
+        <origin xyz="0.55 0.5363 0.35" rpy="${0.0 * deg_to_rad} ${50.0 * deg_to_rad} ${-90.0 * deg_to_rad}"/>
         <origin xyz="0 0 0" rpy="${-90 * deg_to_rad} ${0 * deg_to_rad} ${-90 * deg_to_rad}" />
     </xacro:kinetic_rgb>
