Commit message: Kinematic alignment: Update gripper length, fix URDF artifacts, and implement PyBullet tossing simulation

File: assets/urdf/sawyer_tabletop_electric.urdf (robot description, URDF)
Before this commit: robot sawyer, 28 links, 27 joints
Links:
- link head: geometry visual mesh filename=../meshes/sawyer_description/meshes/sawyer_pv/head.DAE
- link right_l0: geometry visual mesh filename=../meshes/sawyer_description/meshes/sawyer_mp3/l0.DAE
- link right_l1: geometry visual mesh filename=../meshes/sawyer_description/meshes/sawyer_mp3/l1.DAE
- link right_l2_2: geometry 
- link right_l3: geometry visual mesh filename=../meshes/sawyer_description/meshes/sawyer_pv/l3.DAE
- link right_l4_2: geometry 
- link right_l5: geometry visual mesh filename=../meshes/sawyer_description/meshes/sawyer_pv/l5.DAE
- link screen: geometry visual box size=0.24 0.14 0.002

File: assets/urdf/sawyer_tabletop_pneumatic.urdf (robot description, URDF)
Before this commit: robot sawyer, 36 links, 35 joints
Links:
- link head: geometry visual mesh filename=../meshes/sawyer_description/meshes/sawyer_pv/head.DAE
- link right_l0: geometry visual mesh filename=../meshes/sawyer_description/meshes/sawyer_mp3/l0.DAE
- link right_l1: geometry visual mesh filename=../meshes/sawyer_description/meshes/sawyer_mp3/l1.DAE
- link right_l2_2: geometry 
- link right_l3: geometry visual mesh filename=../meshes/sawyer_description/meshes/sawyer_pv/l3.DAE
- link right_l4_2: geometry 
- link right_l5: geometry visual mesh filename=../meshes/sawyer_description/meshes/sawyer_pv/l5.DAE
- link screen: geometry visual box size=0.24 0.14 0.002
