Commit message: Finalizing tossing optimization and simulation improvements: Refined task-space search, MuJoCo/PyBullet visual fixes, and optimized pick-and-toss sequence.

File: assets/urdf/pneumatic_gripper.urdf (robot description, URDF)
Before this commit: robot end_effector, 17 links, 17 joints
Links:
- link right_adapter_bottom: geometry collision cylinder length=0.018 radius=0.046; visual mesh filename=/home/fausto/Projects/sawyer/tossingbot/assets/meshes/tossi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 scale=0.001 0.001 0.001
- link right_adapter_top: geometry collision cylinder length=0.013 radius=0.046; visual mesh filename=/home/fausto/Projects/sawyer/tossingbot/assets/meshes/tossi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 scale=0.001 0.001 0.001
- link right_connector_plate_base: geometry collision cylinder length=0.032 radius=0.06; visual mesh filename=/home/fausto/Projects/sawyer/tossingbot/assets/meshes/tossi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 scale=0.001 0.001 0.001
- link right_ft_sensor_link: geometry collision cylinder length=0.033 radius=0.046; visual mesh filename=/home/fausto/Projects/sawyer/tossingbot/assets/meshes/tossi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 scale=0.001 0.001 0.001
- link right_gripper_l_finger: geometry visual mesh filename=/home/fausto/Projects/sawyer/tossingbot/assets/meshes/tossi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 scale=0.001 0.001 0.001
- link right_gripper_l_finger_base: geometry visual mesh filename=/home/fausto/Projects/sawyer/tossingbot/assets/meshes/tossi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 scale=0.001 0.001 0.001
- link right_gripper_l_finger_body: geometry visual mesh filename=/home/fausto/Projects/sawyer/tossingbot/assets/meshes/tossi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 scale=0.001 0.001 0.001
- link right_gripper_l_pad: geometry collision mesh filename=/home/fausto/Projects/sawyer/tossingbot/assets/meshes/tossi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 scale=0.001 0.001 0.001; visual mesh filename=/home/fausto/Projects/sawyer/tossingbot/assets/meshes/tossi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 scale=0.001 0.001 0.001
- link right_gripper_r_finger: geometry visual mesh filename=/home/fausto/Projects/sawyer/tossingbot/assets/meshes/tossi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 scale=0.001 0.001 0.001
- link right_gripper_r_finger_base: geometry visual mesh filename=/home/fausto/Projects/sawyer/tossingbot/assets/meshes/tossi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 scale=0.001 0.001 0.001
- link right_gripper_r_finger_body: geometry visual mesh filename=/home/fausto/Projects/sawyer/tossingbot/assets/meshes/tossi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 scale=0.001 0.001 0.001
- link right_gripper_r_pad: geometry collision mesh filename=/home/fausto/Projects/sawyer/tossingbot/assets/meshes/tossi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 scale=0.001 0.001 0.001; visual mesh filename=/home/fausto/Projects/sawyer/tossingbot/assets/meshes/tossi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 scale=0.001 0.001 0.001
- link right_pneumatic_gripper_base: geometry collision box size=0.056 0.0871 0.0392; visual mesh filename=/home/fausto/Projects/sawyer/tossingbot/assets/meshes/tossi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 scale=0.001 0.001 0.001
- link right_pneumatic_gripper_cover: geometry visual mesh filename=/home/fausto/Projects/sawyer/tossingbot/assets/meshes/tossi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 scale=0.001 0.001 0.001

File: assets/urdf/sawyer_arm.urdf (robot description, URDF)
Before this commit: robot sawyer, 24 links, 23 joints
Links:
- link head: geometry collision sphere radius=0.18; visual mesh filename=/home/fausto/Projects/sawyer/tossingbot/assets/meshes/sawye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
- link pedestal: geometry collision cylinder length=0.62 radius=0.18; visual mesh filename=/home/fausto/Projects/sawyer/tossingbot/assets/meshes/sawye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
- link right_arm_base_link: geometry collision cylinder length=0.24 radius=0.08; visual mesh filename=/home/fausto/Projects/sawyer/tossingbot/assets/meshes/sawye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
- link right_l0: geometry collision sphere radius=0.07; visual mesh filename=/home/fausto/Projects/sawyer/tossingbot/assets/meshes/sawye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
- link right_l1: geometry collision sphere radius=0.07; visual mesh filename=/home/fausto/Projects/sawyer/tossingbot/assets/meshes/sawye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
- link right_l2: geometry collision cylinder length=0.34 radius=0.06; visual mesh filename=/home/fausto/Projects/sawyer/tossingbot/assets/meshes/sawye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
- link right_l3: geometry collision sphere radius=0.06; visual mesh filename=/home/fausto/Projects/sawyer/tossingbot/assets/meshes/sawye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
- link right_l4: geometry collision cylinder length=0.30 radius=0.045; visual mesh filename=/home/fausto/Projects/sawyer/tossingbot/assets/meshes/sawye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
- link right_l5: geometry collision sphere radius=0.06; visual mesh filename=/home/fausto/Projects/sawyer/tossingbot/assets/meshes/sawye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
- link right_l6: geometry collision cylinder length=0.05 radius=0.055; visual mesh filename=/home/fausto/Projects/sawyer/tossingbot/assets/meshes/sawye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

File: assets/urdf/sawyer_arm_only.urdf (robot description, URDF)
Before this commit: robot sawyer_arm_only, 19 links, 18 joints
Links:
- link head: geometry collision sphere radius=0.18; visual mesh filename=/home/fausto/Projects/sawyer/tossingbot/assets/meshes/sawye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
- link right_arm_base_link: geometry collision cylinder length=0.24 radius=0.08; visual mesh filename=/home/fausto/Projects/sawyer/tossingbot/assets/meshes/sawye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
- link right_l0: geometry collision sphere radius=0.07; visual mesh filename=/home/fausto/Projects/sawyer/tossingbot/assets/meshes/sawye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
- link right_l1: geometry collision sphere radius=0.07; visual mesh filename=/home/fausto/Projects/sawyer/tossingbot/assets/meshes/sawye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
- link right_l2: geometry collision cylinder length=0.34 radius=0.06; visual mesh filename=/home/fausto/Projects/sawyer/tossingbot/assets/meshes/sawye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
- link right_l3: geometry collision sphere radius=0.06; visual mesh filename=/home/fausto/Projects/sawyer/tossingbot/assets/meshes/sawye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
- link right_l4: geometry collision cylinder length=0.30 radius=0.045; visual mesh filename=/home/fausto/Projects/sawyer/tossingbot/assets/meshes/sawye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
- link right_l5: geometry collision sphere radius=0.06; visual mesh filename=/home/fausto/Projects/sawyer/tossingbot/assets/meshes/sawye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
- link right_l6: geometry collision cylinder length=0.05 radius=0.055; visual mesh filename=/home/fausto/Projects/sawyer/tossingbot/assets/meshes/sawye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

File: assets/urdf/sawyer_electric_gripper.urdf (robot description, URDF)
Before this commit: robot end_effector, 9 links, 9 joints
Links:
- link right_connector_plate_base: geometry collision cylinder length=0.0302 radius=0.04; visual mesh filename=/home/fausto/Projects/sawyer/tossingbot/assets/meshes/inter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
- link right_electric_gripper_base: geometry collision cylinder length=0.1 radius=0.029; visual mesh filename=/home/fausto/Projects/sawyer/tossingbot/assets/meshes/inter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
- link right_gripper_l_finger: geometry collision box size=0.01 0.0135 0.075; collision box size=0.01 0.05 0.017
- link right_gripper_l_finger_tip: geometry collision box size=0.016 0.007 0.037; visual mesh filename=/home/fausto/Projects/sawyer/tossingbot/assets/meshes/inter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
- link right_gripper_r_finger: geometry collision box size=0.01 0.0135 0.075; collision box size=0.01 0.05 0.017
- link right_gripper_r_finger_tip: geometry collision box size=0.016 0.007 0.037; visual mesh filename=/home/fausto/Projects/sawyer/tossingbot/assets/meshes/inter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

File: assets/urdf/sawyer_pedestal.urdf (robot description, URDF)
Before this commit: robot sawyer_pedestal, 5 links, 4 joints
Links:
- link pedestal: geometry collision cylinder length=0.62 radius=0.18; visual mesh filename=/home/fausto/Projects/sawyer/tossingbot/assets/meshes/sawye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

File: assets/urdf/sawyer_tabletop_pneumatic.urdf (robot description, URDF)
Before this commit: robot sawyer, 36 links, 35 joints
Links:
- removed link right_l1_2
- removed link right_l2_2
- removed link right_l4_2
- link head: geometry visual mesh filename=/home/fausto/Projects/robosuite/robosuite/models/assets/rob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; visual mesh filename=/home/fausto/Projects/robosuite/robosuite/models/assets/rob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
- link head_camera: mass None -> 1e-04
- link right_adapter_bottom: geometry visual mesh filename=/home/fausto/Projects/sawyer/tossingbot/assets/meshes/tossi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 scale=0.001 0.001 0.001
- link right_adapter_top: geometry visual mesh filename=/home/fausto/Projects/sawyer/tossingbot/assets/meshes/tossi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 scale=0.001 0.001 0.001
- link right_arm_base_link: geometry visual mesh filename=/home/fausto/Projects/robosuite/robosuite/models/assets/rob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; visual mesh filename=/home/fausto/Projects/robosuite/robosuite/models/assets/rob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
- link right_connector_plate_base: geometry visual mesh filename=/home/fausto/Projects/sawyer/tossingbot/assets/meshes/tossi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 scale=0.001 0.001 0.001
- link right_connector_plate_mount: mass None -> 1e-04
- link right_ft_sensor_link: geometry visual mesh filename=/home/fausto/Projects/sawyer/tossingbot/assets/meshes/tossi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 scale=0.001 0.001 0.001
- link right_gripper_l_finger: geometry visual mesh filename=/home/fausto/Projects/sawyer/tossingbot/assets/meshes/tossi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 scale=0.001 0.001 0.001
- link right_gripper_l_finger_base: geometry visual mesh filename=/home/fausto/Projects/sawyer/tossingbot/assets/meshes/tossi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 scale=0.001 0.001 0.001
- link right_gripper_l_finger_body: geometry visual mesh filename=/home/fausto/Projects/sawyer/tossingbot/assets/meshes/tossi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 scale=0.001 0.001 0.001
- link right_gripper_l_pad: geometry collision mesh filename=/home/fausto/Projects/sawyer/tossingbot/assets/meshes/tossi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 scale=0.001 0.001 0.001; visual mesh filename=/home/fausto/Projects/sawyer/tossingbot/assets/meshes/tossi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 scale=0.001 0.001 0.001
- link right_gripper_r_finger: geometry visual mesh filename=/home/fausto/Projects/sawyer/tossingbot/assets/meshes/tossi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 scale=0.001 0.001 0.001
- link right_gripper_r_finger_base: geometry visual mesh filename=/home/fausto/Projects/sawyer/tossingbot/assets/meshes/tossi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 scale=0.001 0.001 0.001
- link right_gripper_r_finger_body: geometry visual mesh filename=/home/fausto/Projects/sawyer/tossingbot/assets/meshes/tossi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 scale=0.001 0.001 0.001
- link right_gripper_r_pad: geometry collision mesh filename=/home/fausto/Projects/sawyer/tossingbot/assets/meshes/tossi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 scale=0.001 0.001 0.001; visual mesh filename=/home/fausto/Projects/sawyer/tossingbot/assets/meshes/tossi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 scale=0.001 0.001 0.001
- link right_gripper_tip: mass None -> 1e-04
- link right_hand: mass 1.0E-08 -> 1e-04; geometry 
- link right_hand_camera: mass None -> 1e-04
- link right_l0: geometry visual mesh filename=/home/fausto/Projects/robosuite/robosuite/models/assets/rob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; visual mesh filename=/home/fausto/Projects/robosuite/robosuite/models/assets/rob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
- link right_l1: geometry visual mesh filename=/home/fausto/Projects/robosuite/robosuite/models/assets/rob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; visual mesh filename=/home/fausto/Projects/robosuite/robosuite/models/assets/rob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
- link right_l2: geometry visual mesh filename=/home/fausto/Projects/robosuite/robosuite/models/assets/rob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; visual mesh filename=/home/fausto/Projects/robosuite/robosuite/models/assets/rob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
- link right_l3: geometry visual mesh filename=/home/fausto/Projects/robosuite/robosuite/models/assets/rob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; visual mesh filename=/home/fausto/Projects/robosuite/robosuite/models/assets/rob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
- link right_l4: geometry visual mesh filename=/home/fausto/Projects/robosuite/robosuite/models/assets/rob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; visual mesh filename=/home/fausto/Projects/robosuite/robosuite/models/assets/rob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
- link right_l5: geometry visual mesh filename=/home/fausto/Projects/robosuite/robosuite/models/assets/rob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; visual mesh filename=/home/fausto/Projects/robosuite/robosuite/models/assets/rob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
- link right_l6: geometry visual mesh filename=/home/fausto/Projects/robosuite/robosuite/models/assets/rob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; visual mesh filename=/home/fausto/Projects/robosuite/robosuite/models/assets/rob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
- link right_pneumatic_gripper_base: geometry visual mesh filename=/home/fausto/Projects/sawyer/tossingbot/assets/meshes/tossi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 scale=0.001 0.001 0.001
- link right_pneumatic_gripper_cover: mass None -> 1e-04; geometry visual mesh filename=/home/fausto/Projects/sawyer/tossingbot/assets/meshes/tossi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 scale=0.001 0.001 0.001
- link right_wrist: mass None -> 1e-04
Joints:
- removed joint attachment_right_hand_to_right_gripper_base
- removed joint right_j1_2
- removed joint right_j2_2
- removed joint right_j4_2
- added joint attachment_to_right_gripper_base: type fixed, parent right_hand, child right_gripper_base, origin xyz=0 0 0 rpy=0 0 0

File: assets/urdf/sawyer_tabletop_pneumatic_clean.urdf (robot description, URDF)
Before this commit: robot sawyer, 25 links, 24 joints
Links:
- removed link right_electric_gripper_base
- removed link right_gripper_l_finger_tip
- removed link right_gripper_r_finger_tip
- added link right_adapter_bottom, mass 0.098; visual mesh filename=/home/fausto/Projects/sawyer/tossingbot/assets/meshes/tossi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 scale=0.001 0.001 0.001
- added link right_adapter_top, mass 0.061; visual mesh filename=/home/fausto/Projects/sawyer/tossingbot/assets/meshes/tossi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 scale=0.001 0.001 0.001
- added link right_ft_sensor_link, mass 0.919; visual mesh filename=/home/fausto/Projects/sawyer/tossingbot/assets/meshes/tossi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 scale=0.001 0.001 0.001
- added link right_gripper_l_finger_base, mass 0.029; visual mesh filename=/home/fausto/Projects/sawyer/tossingbot/assets/meshes/tossi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 scale=0.001 0.001 0.001
- added link right_gripper_l_finger_body, mass 0.037; visual mesh filename=/home/fausto/Projects/sawyer/tossingbot/assets/meshes/tossi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 scale=0.001 0.001 0.001
- added link right_gripper_l_pad, mass 0.040; collision mesh filename=pneumatic_finger_tip.STL scale=0.001 0.001 0.001; visual mesh filename=pneumatic_finger_tip.STL scale=0.001 0.001 0.001
- added link right_gripper_r_finger_base, mass 0.029; visual mesh filename=/home/fausto/Projects/sawyer/tossingbot/assets/meshes/tossi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 scale=0.001 0.001 0.001
- added link right_gripper_r_finger_body, mass 0.037; visual mesh filename=/home/fausto/Projects/sawyer/tossingbot/assets/meshes/tossi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 scale=0.001 0.001 0.001
- added link right_gripper_r_pad, mass 0.040; collision mesh filename=pneumatic_finger_tip.STL scale=0.001 0.001 0.001; visual mesh filename=pneumatic_finger_tip.STL scale=0.001 0.001 0.001
- added link right_l1_2, mass 1e-04
- added link right_l2_2, mass 1e-04
- added link right_l4_2, mass 1e-04
- added link right_pneumatic_gripper_base, mass 0.311; visual mesh filename=/home/fausto/Projects/sawyer/tossingbot/assets/meshes/tossi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 scale=0.001 0.001 0.001
- added link right_pneumatic_gripper_cover, mass 1e-04; visual mesh filename=/home/fausto/Projects/sawyer/tossingbot/assets/meshes/tossi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 scale=0.001 0.001 0.001
- link right_connector_plate_base: mass 1e-04 -> 0.387; geometry visual mesh filename=/home/fausto/Projects/sawyer/tossingbot/assets/meshes/tossi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 scale=0.001 0.001 0.001
- link right_gripper_base: mass 0.47 -> 1.902
- link right_gripper_l_finger: mass 0.001 -> 0.010; geometry visual mesh filename=/home/fausto/Projects/sawyer/tossingbot/assets/meshes/tossi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 scale=0.001 0.001 0.001
- link right_gripper_r_finger: mass 0.001 -> 0.010; geometry visual mesh filename=/home/fausto/Projects/sawyer/tossingbot/assets/meshes/tossi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 scale=0.001 0.001 0.001
- link screen: geometry 
Joints:
- removed joint right_electric_gripper_base_joint
- removed joint right_gripper_l_finger_tip_joint
- removed joint right_gripper_r_finger_tip_joint
- added joint right_adapter_top_bottom_joint: type fixed, parent right_adapter_top, child right_adapter_bottom, origin xyz=0 0 0.013 rpy=0 0 0
- added joint right_connector_plate_ft_sensor_joint: type fixed, parent right_connector_plate_mount, child right_ft_sensor_link, origin xyz=0 0 0 rpy=0 0 0
- added joint right_ft_sensor_adapter_top_joint: type fixed, parent right_ft_sensor_link, child right_adapter_top, origin xyz=0 0 0.033 rpy=0 0 0
- added joint right_gripper_l_finger_base_joint: type fixed, parent right_gripper_l_finger, child right_gripper_l_finger_base, origin xyz=0 0 0.012 rpy=0 0 0
- added joint right_gripper_l_finger_body_joint: type fixed, parent right_gripper_l_finger_base, child right_gripper_l_finger_body, origin xyz=0 0.024 0.006 rpy=0 0 0
- added joint right_gripper_l_pad_joint: type fixed, parent right_gripper_l_finger_body, child right_gripper_l_pad, origin xyz=0 0 0 rpy=0 0 0
- added joint right_gripper_r_finger_base_joint: type fixed, parent right_gripper_r_finger, child right_gripper_r_finger_base, origin xyz=0 0 0.012 rpy=0 0 0
- added joint right_gripper_r_finger_body_joint: type fixed, parent right_gripper_r_finger_base, child right_gripper_r_finger_body, origin xyz=0 -0.024 0.006 rpy=0 0 0
- added joint right_gripper_r_pad_joint: type fixed, parent right_gripper_r_finger_body, child right_gripper_r_pad, origin xyz=0 0 0 rpy=0 0 0
- added joint right_j1_2: type fixed, parent right_l1, child right_l1_2, origin xyz=0 0 0 rpy=0 0 0, axis 0 0 1
- added joint right_j2_2: type fixed, parent right_l2, child right_l2_2, origin xyz=0 0 0 rpy=0 0 0, axis 0 0 1
- added joint right_j4_2: type fixed, parent right_l4, child right_l4_2, origin xyz=0 0 0 rpy=0 0 0, axis 0 0 1
- added joint right_pneumatic_base_joint: type fixed, parent right_adapter_bottom, child right_pneumatic_gripper_base, origin xyz=0 0 0.018 rpy=0 0 0
- added joint right_pneumatic_cover_joint: type fixed, parent right_adapter_bottom, child right_pneumatic_gripper_cover, origin xyz=0 0 0.018 rpy=0 0 0
- joint right_connector_plate_mount_joint: origin xyz=0 0 0.0176 rpy=0 0 0 -> xyz=0 0 0.032  rpy=0 0 0
- joint right_gripper_l_finger_joint: limit lower=0.0 upper=0.020833 effort=20.0 velocity=5.0 -> lower=0.0 upper=0.016 effort=20.0 velocity=5.0; origin xyz=0.003 -0.0014999999999999996 0.04552 rpy=0 0 0 -> xyz=0 0 0.0282 rpy=0 0 0; parent right_electric_gripper_base -> right_pneumatic_gripper_base
- joint right_gripper_r_finger_joint: limit lower=-0.020833 upper=0.0 effort=20.0 velocity=5.0 -> lower=-0.016 upper=0.0 effort=20.0 velocity=5.0; origin xyz=0.003 0.0014999999999999996 0.04552 rpy=0 0 0 -> xyz=0 0 0.0282 rpy=0 0 0; parent right_electric_gripper_base -> right_pneumatic_gripper_base
- joint right_gripper_tip_joint: origin xyz=0 0 0.14062 rpy=0 0 0 -> xyz=0 0 0.2088 rpy=0 0 0

File: assets/urdf/sawyer_tabletop_pneumatic_pybullet.urdf (robot description, URDF)
Before this commit: robot sawyer, 41 links, 41 joints
Links:
- removed link base
- removed link controller_box
- removed link pedestal
- removed link pedestal_feet
- removed link right_l1_2
- removed link right_l2_2
- removed link right_l4_2
- removed link torso
- link head: geometry visual mesh filename=/home/fausto/Projects/sawyer/tossingbot/assets/meshes/sawye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
- link head_camera: mass None -> 1e-04
- link right_adapter_bottom: geometry visual mesh filename=/home/fausto/Projects/sawyer/tossingbot/assets/meshes/tossi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 scale=0.001 0.001 0.001
- link right_adapter_top: geometry visual mesh filename=/home/fausto/Projects/sawyer/tossingbot/assets/meshes/tossi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 scale=0.001 0.001 0.001
- link right_arm_base_link: geometry visual mesh filename=/home/fausto/Projects/sawyer/tossingbot/assets/meshes/sawye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
- link right_connector_plate_base: geometry visual mesh filename=/home/fausto/Projects/sawyer/tossingbot/assets/meshes/tossi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 scale=0.001 0.001 0.001
- link right_connector_plate_mount: mass None -> 1e-04
- link right_ft_sensor_link: geometry visual mesh filename=/home/fausto/Projects/sawyer/tossingbot/assets/meshes/tossi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 scale=0.001 0.001 0.001
- link right_gripper_tip: mass None -> 1e-04
- link right_hand: mass 1.0E-08 -> 1e-04; geometry 
- link right_hand_camera: mass None -> 1e-04
- link right_l0: geometry visual mesh filename=/home/fausto/Projects/sawyer/tossingbot/assets/meshes/sawye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
- link right_l1: geometry visual mesh filename=/home/fausto/Projects/sawyer/tossingbot/assets/meshes/sawye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
- link right_l2: geometry visual mesh filename=/home/fausto/Projects/sawyer/tossingbot/assets/meshes/sawye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
- link right_l3: geometry visual mesh filename=/home/fausto/Projects/sawyer/tossingbot/assets/meshes/sawye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
- link right_l4: geometry visual mesh filename=/home/fausto/Projects/sawyer/tossingbot/assets/meshes/sawye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
- link right_l5: geometry visual mesh filename=/home/fausto/Projects/sawyer/tossingbot/assets/meshes/sawye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
- link right_l6: geometry visual mesh filename=/home/fausto/Projects/sawyer/tossingbot/assets/meshes/sawye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
- link right_pneumatic_gripper_base: geometry visual mesh filename=/home/fausto/Projects/sawyer/tossingbot/assets/meshes/tossi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 scale=0.001 0.001 0.001
- link right_pneumatic_gripper_cover: mass None -> 1e-04
- link right_wrist: mass None -> 1e-04
- link screen: geometry visual box size=0.24 0.14 0.002
Joints:
- removed joint attachment_joint
- removed joint controller_box_fixed
- removed joint pedestal_feet_fixed
- removed joint pedestal_fixed
- removed joint right_arm_mount
- removed joint right_gripper_base_joint
- removed joint right_j1_2
- removed joint right_j2_2
- removed joint right_j4_2
- removed joint torso_t0
- added joint attachment_to_right_gripper_base: type fixed, parent right_hand, child right_gripper_base, origin xyz=0 0 0 rpy=0 0 0

File: assets/urdf/sawyer_with_electric.urdf (robot description, URDF)
Before this commit: robot sawyer, 33 links, 32 joints
Links:
- link head: geometry collision sphere radius=0.18; visual mesh filename=/home/fausto/Projects/sawyer/tossingbot/assets/meshes/sawye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
- link pedestal: geometry collision cylinder length=0.62 radius=0.18; visual mesh filename=/home/fausto/Projects/sawyer/tossingbot/assets/meshes/sawye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
- link right_arm_base_link: geometry collision cylinder length=0.24 radius=0.08; visual mesh filename=/home/fausto/Projects/sawyer/tossingbot/assets/meshes/sawye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
- link right_connector_plate_base: geometry collision cylinder length=0.0302 radius=0.04; visual mesh filename=/home/fausto/Projects/sawyer/tossingbot/assets/meshes/inter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
- link right_electric_gripper_base: geometry collision cylinder length=0.1 radius=0.029; visual mesh filename=/home/fausto/Projects/sawyer/tossingbot/assets/meshes/inter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
- link right_gripper_l_finger: geometry collision box size=0.01 0.0135 0.075; collision box size=0.01 0.05 0.017
- link right_gripper_l_finger_tip: geometry collision box size=0.016 0.007 0.037; visual mesh filename=/home/fausto/Projects/sawyer/tossingbot/assets/meshes/inter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
- link right_gripper_r_finger: geometry collision box size=0.01 0.0135 0.075; collision box size=0.01 0.05 0.017
- link right_gripper_r_finger_tip: geometry collision box size=0.016 0.007 0.037; visual mesh filename=/home/fausto/Projects/sawyer/tossingbot/assets/meshes/inter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
- link right_l0: geometry collision sphere radius=0.07; visual mesh filename=/home/fausto/Projects/sawyer/tossingbot/assets/meshes/sawye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
- link right_l1: geometry collision sphere radius=0.07; visual mesh filename=/home/fausto/Projects/sawyer/tossingbot/assets/meshes/sawye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
- link right_l2: geometry collision cylinder length=0.34 radius=0.06; visual mesh filename=/home/fausto/Projects/sawyer/tossingbot/assets/meshes/sawye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
- link right_l3: geometry collision sphere radius=0.06; visual mesh filename=/home/fausto/Projects/sawyer/tossingbot/assets/meshes/sawye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
- link right_l4: geometry collision cylinder length=0.30 radius=0.045; visual mesh filename=/home/fausto/Projects/sawyer/tossingbot/assets/meshes/sawye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
- link right_l5: geometry collision sphere radius=0.06; visual mesh filename=/home/fausto/Projects/sawyer/tossingbot/assets/meshes/sawye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
- link right_l6: geometry collision cylinder length=0.05 radius=0.055; visual mesh filename=/home/fausto/Projects/sawyer/tossingbot/assets/meshes/sawye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
