Commit message: Finalizing tossing optimization and simulation improvements: Refined task-space search, MuJoCo/PyBullet visual fixes, and optimized pick-and-toss sequence.

File: assets/urdf/sawyer_with_pneumatic.urdf (robot description, URDF)
Before this commit: robot sawyer, 41 links, 40 joints
Links:
- link head: geometry collision sphere radius=0.18; visual mesh filename=/home/fausto/Projects/sawyer/tossingbot/assets/meshes/sawye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
- link pedestal: geometry collision cylinder length=0.62 radius=0.18; visual mesh filename=/home/fausto/Projects/sawyer/tossingbot/assets/meshes/sawye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
- link right_adapter_bottom: geometry collision cylinder length=0.018 radius=0.046; visual mesh filename=/home/fausto/Projects/sawyer/tossingbot/assets/meshes/tossi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 scale=0.001 0.001 0.001
- link right_adapter_top: geometry collision cylinder length=0.013 radius=0.046; visual mesh filename=/home/fausto/Projects/sawyer/tossingbot/assets/meshes/tossi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 scale=0.001 0.001 0.001
- link right_arm_base_link: geometry collision cylinder length=0.24 radius=0.08; visual mesh filename=/home/fausto/Projects/sawyer/tossingbot/assets/meshes/sawye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
- link right_connector_plate_base: geometry collision cylinder length=0.032 radius=0.06; visual mesh filename=/home/fausto/Projects/sawyer/tossingbot/assets/meshes/tossi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 scale=0.001 0.001 0.001
- link right_ft_sensor_link: geometry collision cylinder length=0.033 radius=0.046; visual mesh filename=/home/fausto/Projects/sawyer/tossingbot/assets/meshes/tossi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 scale=0.001 0.001 0.001
- link right_gripper_l_finger: geometry visual mesh filename=/home/fausto/Projects/sawyer/tossingbot/assets/meshes/tossi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 scale=0.001 0.001 0.001
- link right_gripper_l_finger_base: geometry visual mesh filename=/home/fausto/Projects/sawyer/tossingbot/assets/meshes/tossi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 scale=0.001 0.001 0.001
- link right_gripper_l_finger_body: geometry visual mesh filename=/home/fausto/Projects/sawyer/tossingbot/assets/meshes/tossi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 scale=0.001 0.001 0.001
- link right_gripper_l_pad: geometry collision mesh filename=/home/fausto/Projects/sawyer/tossingbot/assets/meshes/tossi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 scale=0.001 0.001 0.001; visual mesh filename=/home/fausto/Projects/sawyer/tossingbot/assets/meshes/tossi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 scale=0.001 0.001 0.001
- link right_gripper_r_finger: geometry visual mesh filename=/home/fausto/Projects/sawyer/tossingbot/assets/meshes/tossi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 scale=0.001 0.001 0.001
- link right_gripper_r_finger_base: geometry visual mesh filename=/home/fausto/Projects/sawyer/tossingbot/assets/meshes/tossi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 scale=0.001 0.001 0.001
- link right_gripper_r_finger_body: geometry visual mesh filename=/home/fausto/Projects/sawyer/tossingbot/assets/meshes/tossi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 scale=0.001 0.001 0.001
- link right_gripper_r_pad: geometry collision mesh filename=/home/fausto/Projects/sawyer/tossingbot/assets/meshes/tossi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 scale=0.001 0.001 0.001; visual mesh filename=/home/fausto/Projects/sawyer/tossingbot/assets/meshes/tossi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 scale=0.001 0.001 0.001
- link right_l0: geometry collision sphere radius=0.07; visual mesh filename=/home/fausto/Projects/sawyer/tossingbot/assets/meshes/sawye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
- link right_l1: geometry collision sphere radius=0.07; visual mesh filename=/home/fausto/Projects/sawyer/tossingbot/assets/meshes/sawye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
- link right_l2: geometry collision cylinder length=0.34 radius=0.06; visual mesh filename=/home/fausto/Projects/sawyer/tossingbot/assets/meshes/sawye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
- link right_l3: geometry collision sphere radius=0.06; visual mesh filename=/home/fausto/Projects/sawyer/tossingbot/assets/meshes/sawye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
- link right_l4: geometry collision cylinder length=0.30 radius=0.045; visual mesh filename=/home/fausto/Projects/sawyer/tossingbot/assets/meshes/sawye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
- link right_l5: geometry collision sphere radius=0.06; visual mesh filename=/home/fausto/Projects/sawyer/tossingbot/assets/meshes/sawye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
- link right_l6: geometry collision cylinder length=0.05 radius=0.055; visual mesh filename=/home/fausto/Projects/sawyer/tossingbot/assets/meshes/sawye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
- link right_pneumatic_gripper_base: geometry collision box size=0.056 0.0871 0.0392; visual mesh filename=/home/fausto/Projects/sawyer/tossingbot/assets/meshes/tossi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 scale=0.001 0.001 0.001
- link right_pneumatic_gripper_cover: geometry visual mesh filename=/home/fausto/Projects/sawyer/tossingbot/assets/meshes/tossi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 scale=0.001 0.001 0.001
